File: USB2LPT_1.7_adapter.brd (EAGLE design)
At the start: 43.2 x 49.5 mm, 27 parts

Commit message: Board routing. Not quite done.
Parts:
- moved R12 31.4 mm to (21.6, 39.6), turned to 180 degrees
- moved R6 22.3 mm to (15.2, 18.0), turned to 0 degrees
- moved R17 17.9 mm to (21.6, 33.3), turned to 180 degrees
- moved R5 16.5 mm to (15.2, 24.1), turned to 0 degrees
- moved R15 13.7 mm to (21.6, 36.3), turned to 180 degrees
- moved R8 12.4 mm to (15.2, 21.1), turned to 0 degrees
- moved R10 10.9 mm to (15.2, 33.0), turned to 0 degrees
- moved R7 10.5 mm to (15.2, 27.2), turned to 0 degrees
- moved R21 10.4 mm to (27.9, 46.7), turned to 0 degrees
- moved R16 9.91 mm to (15.2, 30.2)
- moved R3 8.29 mm to (21.6, 18.0), turned to 180 degrees
- moved Q1 7.69 mm to (17.8, 43.4), turned to 180 degrees
- moved R14 6.67 mm to (21.6, 30.0), turned to 180 degrees
- moved R20 4.72 mm to (17.8, 47.2), turned to 0 degrees
- moved R11 4.57 mm to (15.2, 36.3)
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Routing:
- net PD4: track 0.00 -> 90.8 mm, vias 0 -> 1
- net PD6: track 0.00 -> 72.0 mm, vias 0 -> 2
- net PB0: track 0.00 -> 68.6 mm, vias 0 -> 3
- net IFCLK: track 0.00 -> 68.2 mm, vias 0 -> 1
- net PD3: track 0.00 -> 68.0 mm, vias 0 -> 2
- net PB1: track 0.00 -> 67.4 mm, vias 0 -> 2
- net PD7: track 0.00 -> 64.6 mm
- net PD5: track 0.00 -> 64.0 mm
- net CTL2: track 0.00 -> 63.9 mm, vias 0 -> 2
- net PB2: track 0.00 -> 60.6 mm, vias 0 -> 2
- net PB3: track 0.00 -> 59.3 mm, vias 0 -> 2
- net PD1: track 0.00 -> 58.1 mm, vias 0 -> 2
- net PD2: track 0.00 -> 56.6 mm, vias 0 -> 2
- net PD0: track 0.00 -> 53.4 mm, vias 0 -> 2
- net +3V3: track 0.00 -> 52.5 mm, vias 0 -> 2
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Other:
- board size 43.2 x 49.5 mm -> 43.4 x 49.5 mm

Commit message: Cleanup PCB some more
Routing:
- net PB2: track 60.6 -> 83.2 mm
- net IFCLK: track 68.2 -> 83.6 mm
- net PB1: track 67.4 -> 81.8 mm
- net PB0: track 68.6 -> 82.8 mm
- net PB3: track 59.3 -> 66.3 mm
- net CTL1: track 46.4 -> 52.1 mm, vias 0 -> 2
- net CTL2: track 63.9 -> 62.8 mm, vias 2 -> 0
- net PD3: track 68.0 -> 68.5 mm, vias 2 -> 0

Commit message: idem
Parts:
- moved R2 4.58 mm to (21.3, 25.7)
- moved R4 4.07 mm to (21.3, 18.8)
- moved R6 3.09 mm to (15.7, 21.1)
- moved R3 3.06 mm to (21.3, 21.1)
- moved R8 2.34 mm to (15.7, 23.4)
- moved R5 1.61 mm to (15.7, 25.7)
- moved R13 1.37 mm to (15.7, 38.4)
- moved R12 1.30 mm to (21.3, 38.4)
- moved R14 0.92 mm to (22.1, 30.7)
- moved R7 0.92 mm to (15.7, 27.9)
- moved R10 0.92 mm to (15.7, 33.8)
- moved R1 0.80 mm to (21.3, 23.4)
- moved R9 0.80 mm to (21.3, 27.9)
- moved R16 0.57 mm to (15.0, 30.7)
- moved R11 0.57 mm to (15.7, 36.1)
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Routing:
- net PULL-UPS: track 54.3 -> 41.8 mm
- net PB2: track 83.2 -> 72.7 mm
- net PB3: track 66.3 -> 74.9 mm
- net PB4: track 34.6 -> 39.7 mm, vias 2 -> 1
- net PD2: track 56.6 -> 60.7 mm
- net PB5: track 34.8 -> 37.8 mm, vias 2 -> 1
- net PB0: track 82.8 -> 79.9 mm
- net PB7: track 41.4 -> 44.2 mm
- net PD5: track 64.0 -> 66.5 mm
- net PD3: track 68.5 -> 70.9 mm
- net PD4: track 90.8 -> 93.0 mm
- net PB6: track 49.6 -> 48.3 mm, vias 2 -> 0
- net PD1: track 58.1 -> 59.3 mm
- net CTL1: track 52.1 -> 51.3 mm
- net PD6: track 72.0 -> 72.7 mm
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
Commit message: idem
Parts:
- removed X4: (no value), con-subd:F25D
- added +5V: CON_HEADER_1X01-PTH_08_17, dp_devices:M1X2_08_17
- added J1: CON_HEADER_1X03-PTH, dp_devices:M1X3
- added U$1: (no value), dp_devices:JUMP3_DESC_LEFT
- added U$5: (no value), dp_devices:JUMP3_DESC_RIGHT
- added X101: (no value), con-lstb:MA10-2
- R1, R2: value 4K7 -> 470
- R12, R6, R8: value 4K7 -> 2K2
- R15, R16, R17: value 2K2 -> 4K7
- R18, R19: value 470 -> 4K7
- X1: device con-lstb:MA10-2 -> con-subd:F25D
- moved X1 33.6 mm to (19.1, 1.47), flipped to the top, turned to 180 degrees
- moved R21 32.7 mm to (21.3, 14.7)
- moved R20 32.2 mm to (10.9, 15.7), turned to 90 degrees
- moved R19 30.6 mm to (21.3, 17.0), turned to 180 degrees
- moved R18 30.4 mm to (21.3, 19.3)
- moved Q1 27.8 mm to (15.6, 15.7), turned to 270 degrees
- moved R1 19.9 mm to (12.4, 41.1), turned to 90 degrees
- moved R4 17.9 mm to (21.3, 36.7)
- moved R13 16.8 mm to (15.7, 21.6)
- moved R3 16.6 mm to (15.7, 36.7), turned to 0 degrees
- moved R2 16.5 mm to (27.7, 40.9), turned to 90 degrees
- moved R17 15.5 mm to (15.7, 19.3), turned to 0 degrees
- moved R6 14.5 mm to (21.3, 34.4), turned to 180 degrees
- moved R15 13.4 mm to (15.7, 23.9), turned to 0 degrees
- moved R12 12.2 mm to (21.3, 26.2)
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- renumbered X2 to X100
Connections:
- new net 5V_PAD: +5V.1, J1.3
- new net VSELECT: J1.2, Q1.2, R20.1
- net +3V3: now also J1.1, X101.12, X101.2; no longer Q1.2, R20.1, X1.12, X1.2
- net CTL0: now also R12.1, X1.1; no longer R9.1, X4.1
- net CTL1: now also R10.1, X1.14; no longer R14.1, X4.14
- net CTL2: now also R8.1, X1.17; no longer R17.1, X4.17
- net GND: now also X1.19, X1.20, X1.24, X1.25, X101.1, X101.11, X101.16, X101.18, X101.9; no longer X1.1, X1.11, X1.16, X1.9, X4.18, X4.19, X4.20, X4.24, X4.25
- net IFCLK: now also R9.1, X1.16, X101.10, X101.15; no longer R16.1, X1.10, X1.15, X4.16
- net N$5: now also R1.2; no longer R18.2
- net N$6: now also R2.2; no longer R19.2
- net PA4: now also R1.1; no longer R18.1
- net PA5: now also R2.1; no longer R19.1
- net PB0: now also R15.1, X1.2, X101.5; no longer R8.1, X1.5, X4.2
- net PB1: now also R11.1, X1.3, X101.6; no longer R7.1, X1.6, X4.3
- net PB2: now also R17.1, X1.4, X101.3; no longer R6.1, X1.3, X4.4
- net PB3: now also R13.1, X1.5, X101.4; no longer R5.1, X1.4, X4.5
- net PB4: now also R19.1, X1.6; no longer R4.1, X4.6
- net PB5: now also R18.1, X1.7; no longer R3.1, X4.7
- net PB6: now also R14.1, X1.8; no longer R2.1, X4.8
- net PB7: now also R16.1, X1.9; no longer R1.1, X4.9
- net PD0: now also X1.21; no longer X4.21
- net PD1: now also X1.22; no longer X4.22
- net PD2: now also X1.23; no longer X4.23
- net PD3: now also R6.1, X1.15; no longer R15.1, X4.15
- net PD4: now also R4.1, X1.13; no longer R12.1, X4.13
- net PD5: now also R5.1, X1.12, X101.19; no longer R11.1, X1.19, X4.12
- net PD6: now also R3.1, X1.10, X101.13, X101.20; no longer R13.1, X1.13, X1.20, X4.10
- net PD7: now also R7.1, X1.11, X101.14, X101.17; no longer R10.1, X1.14, X1.17, X4.11
- net PULL-UPS: now also R18.2, R19.2; no longer R1.2, R2.2
- net SCL: now also X101.7; no longer X1.7
- net SDA: now also X101.8; no longer X1.8
Routing:
- net VSELECT: track 0.00 -> 39.4 mm, vias 0 -> 1
- net +3V3: track 52.5 -> 28.4 mm, vias 2 -> 1
- net PA4: track 49.5 -> 29.0 mm, vias 1 -> 2
- net PD0: track 53.9 -> 41.8 mm
- net PD1: track 59.3 -> 48.3 mm
- net PD2: track 60.7 -> 49.8 mm
- net PA6: track 18.3 -> 28.8 mm, vias 0 -> 1
- net PB1: track 82.0 -> 72.5 mm
- net PB0: track 79.9 -> 71.2 mm
- net CTL2: track 62.8 -> 54.6 mm
- net CTL1: track 51.3 -> 43.8 mm
- net PB3: track 74.9 -> 67.6 mm
- net PD5: track 66.5 -> 59.6 mm
- net PD7: track 64.8 -> 57.9 mm
- net PD6: track 72.7 -> 66.0 mm
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- removed copper zone on layer 1, net GND
Other:
- board size 43.4 x 49.5 mm -> 41.4 x 41.4 mm
- board text added: "+3.3V IOs"
- board text added: "+5V IOs"
- board text added: "+5V in"
- board text added: "1"
- board text added: "13"
- board text added: "14"
- board text added: "20"
- board text added: "25"
- board text added: "Connect to host board +5Vdc source"
- board text removed: "Rev: 1.0"

Commit message: Final revision of the board Added Gerber archive
Parts:
- removed J1: CON_HEADER_1X03-PTH, dp_devices:M1X3
- removed LED2: (no value), dp_devices:LED-805
- added HI-SPEED: (no value), dp_devices:LED-805
- added VSELECT: VSELECT_HEADER, parts:HEADER_1X3
- R10: value 4K7 -> 2K2
- R6: value 2K2 -> 4K7
- moved R2 2.54 mm to (25.1, 40.9), turned to 270 degrees
- moved R13 2.29 mm to (15.7, 23.9)
- moved R15 2.29 mm to (15.7, 21.6)
- renumbered LED1 to ACTIVITY, U$5 to $$U$2
Connections:
- removed net N$6: LED2.C, R2.2
- new net N$1: HI-SPEED.A, R2.1
- net +3V3: now also R2.2, VSELECT.1; no longer J1.1, LED2.A
- net 5V_PAD: now also VSELECT.3; no longer J1.3
- net PA5: now also HI-SPEED.C; no longer R2.1
- net PB0: now also R13.1; no longer R15.1
- net PB3: now also R15.1; no longer R13.1
- net VSELECT: now also VSELECT.2; no longer J1.2
Routing:
- net PD6: track 66.0 -> 139.1 mm
- net IFCLK: track 76.6 -> 144.4 mm
- net PD0: track 41.8 -> 99.8 mm
- net PB0: track 71.2 -> 128.9 mm
- net PD2: track 49.8 -> 101.3 mm
- net PB5: track 32.5 -> 82.3 mm
- net CTL2: track 54.6 -> 103.8 mm
- net PD1: track 48.3 -> 95.2 mm
- net +3V3: track 28.4 -> 73.8 mm
- net PA4: track 29.0 -> 73.6 mm
- net PB4: track 34.8 -> 78.4 mm
- net CTL1: track 43.8 -> 84.8 mm
- net PD7: track 57.9 -> 95.3 mm
- net PB2: track 66.2 -> 100.5 mm
- net PB3: track 67.6 -> 101.5 mm
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Other:
- board text added: "+3.3V IO"
- board text added: "+5V IO"
- board text added: "Original work by Henrik Haftmann"
- board text added: "USB2LPT 1.7 adapter v1.0 Benjamin Fiset-Deschênes www.benjaminfd.com Licensed under GPLv3"
- board text removed: "+3.3V IOs"
- board text removed: "+5V IOs"
- board text removed: "20"
