File: USB2LPT_1.7_adapter.sch (EAGLE design)
At the start: 27 parts

Commit message: idem
Parts:
- removed X4: (no value), con-subd:F25D
- added +5V: CON_HEADER_1X01-PTH_08_17, dp_devices:CON_HEADER_1X01-PTH_08_17
- added J1: CON_HEADER_1X03-PTH, dp_devices:CON_HEADER_1X03-PTH
- added X101: (no value), con-lstb:MA10-2
- R1, R2: value 4K7 -> 470
- R12, R6, R8: value 4K7 -> 2K2
- R15, R16, R17: value 2K2 -> 4K7
- R18, R19: value 470 -> 4K7
- X1: device con-lstb:MA10-2 -> con-subd:F25D
- renumbered X2 to X100
Connections:
- new net 5V_PAD: +5V.1, J1.3
- new net VSELECT: J1.2, Q1.E, R20.1
- net +3V3: now also J1.1, X101.12, X101.2; no longer Q1.E, R20.1, X1.12, X1.2
- net CTL0: now also R12.1, X1.1; no longer R9.1, X4.1
- net CTL1: now also R10.1, X1.14; no longer R14.1, X4.14
- net CTL2: now also R8.1, X1.17; no longer R17.1, X4.17
- net GND: now also X1.19, X1.20, X1.24, X1.25, X101.1, X101.11, X101.16, X101.18, X101.9; no longer X1.1, X1.11, X1.16, X1.9, X4.18, X4.19, X4.20, X4.24, X4.25
- net IFCLK: now also R9.1, X1.16, X101.10, X101.15; no longer R16.1, X1.10, X1.15, X4.16
- net N$5: now also R1.2; no longer R18.2
- net N$6: now also R2.2; no longer R19.2
- net PA4: now also R1.1; no longer R18.1
- net PA5: now also R2.1; no longer R19.1
- net PB0: now also R15.1, X1.2, X101.5; no longer R8.1, X1.5, X4.2
- net PB1: now also R11.1, X1.3, X101.6; no longer R7.1, X1.6, X4.3
- net PB2: now also R17.1, X1.4, X101.3; no longer R6.1, X1.3, X4.4
- net PB3: now also R13.1, X1.5, X101.4; no longer R5.1, X1.4, X4.5
- net PB4: now also R19.1, X1.6; no longer R4.1, X4.6
- net PB5: now also R18.1, X1.7; no longer R3.1, X4.7
- net PB6: now also R14.1, X1.8; no longer R2.1, X4.8
- net PB7: now also R16.1, X1.9; no longer R1.1, X4.9
- net PD0: now also X1.21; no longer X4.21
- net PD1: now also X1.22; no longer X4.22
- net PD2: now also X1.23; no longer X4.23
- net PD3: now also R6.1, X1.15; no longer R15.1, X4.15
- net PD4: now also R4.1, X1.13; no longer R12.1, X4.13
- net PD5: now also R5.1, X1.12, X101.19; no longer R11.1, X1.19, X4.12
- net PD6: now also R3.1, X1.10, X101.13, X101.20; no longer R13.1, X1.13, X1.20, X4.10
- net PD7: now also R7.1, X1.11, X101.14, X101.17; no longer R10.1, X1.14, X1.17, X4.11
- net PULL-UPS: now also R18.2, R19.2; no longer R1.2, R2.2
- net SCL: now also X101.7; no longer X1.7
- net SDA: now also X101.8; no longer X1.8
Other:
- moved on the sheet: R1, R10, R11, R12, R13, R14, R15, R16, R17, R18, R19, R2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

Commit message: Final revision of the board Added Gerber archive
Parts:
- removed J1: CON_HEADER_1X03-PTH, dp_devices:CON_HEADER_1X03-PTH
- removed LED1, LED2: (no value), dp_devices:LED-0805
- added ACTIVITY, HI-SPEED: (no value), dp_devices:LED-0805
- added VSELECT: VSELECT_HEADER, parts:VSELECT_HEADER
- R10: value 4K7 -> 2K2
- R6: value 2K2 -> 4K7
Connections:
- removed net N$6: LED2.C, R2.2
- new net N$1: HI-SPEED.A, R2.1
- net +3V3: now also ACTIVITY.A, R2.2, VSELECT.1; no longer J1.1, LED1.A, LED2.A
- net 5V_PAD: now also VSELECT.3; no longer J1.3
- net N$5: now also ACTIVITY.C; no longer LED1.C
- net PA5: now also HI-SPEED.C; no longer R2.1
- net PB0: now also R13.1; no longer R15.1
- net PB3: now also R15.1; no longer R13.1
- net VSELECT: now also VSELECT.2; no longer J1.2
Other:
- moved on the sheet: Q1, R1, R10, R11, R12, R13, R14, R15, R16, R17, R18, R19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
